File: PushGame/MainBoard.kicad_pcb (KiCad board)
At the start: 2 copper layers, 25 parts, among them Q1 BC337, Q2 BC337, Q3 BC337, Q4 BC337, Q5 BC337, Q6 BC337, Q7 BC337, Q8 BC337, Q9 BC337, U1 LM7805_TO220

Commit message: Add files via upload
Other:
- board outline added: 136.5 x 45 mm
Changed lines of the file:
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@@
 	)
 	(gr_rect
-		(start 108 39.5)
-		(end 247 82.5)
+		(start 111.5 38.5)
+		(end 248 83.5)
 		(stroke
-			(width 0.2)
-			(type solid)
+			(width 0.05)
+			(type default)
 		)
 		(fill no)
-		(layer "B.Cu")
+		(layer "Edge.Cuts")
 	)
 	(gr_text "P5"
@@
 		(polygon
 			(pts
-				(xy 108 39.5) (xy 247 39.5) (xy 247 82.5) (xy 108 82.5)
-			)
-		)
+				(xy 112.5 39.5) (xy 247 39.5) (xy 247 82.5) (xy 112.5 82.5)
+			)
+		)
